File: pulsarPCB/pulsarPCB.kicad_pcb (KiCad board)
At the start: 2 copper layers, 11 parts, among them Q1 IRLR3110Z

Commit message: change topology
Parts:
- added C10: 100n, Capacitor_SMD:C_1210_3225Metric, F.Cu at (230.8, 83.6)
- added C11: 100n, Capacitor_SMD:C_0603_1608Metric, F.Cu at (226.0, 78.5)
- added C12: 100n, Capacitor_SMD:C_0603_1608Metric, F.Cu at (226.0, 81.0)
- added C13: 4u7, Capacitor_SMD:C_1206_3216Metric, F.Cu at (221.1, 85.6)
- added C14: 100n, Capacitor_SMD:C_1206_3216Metric, F.Cu at (221.1, 88.9)
- added C15: 100n, Capacitor_SMD:C_1206_3216Metric, F.Cu at (221.1, 92.3)
- added C16: 1u, Capacitor_SMD:C_0603_1608Metric, F.Cu at (226.0, 83.5)
- added C17: 1u, Capacitor_SMD:C_0603_1608Metric, F.Cu at (226.0, 86.0)
- added C18: 1u, Capacitor_SMD:C_0603_1608Metric, F.Cu at (226.0, 88.5)
- added C19: 100n, Capacitor_SMD:C_1210_3225Metric, F.Cu at (230.8, 87.8)
- added C20: 100n, Capacitor_SMD:C_1210_3225Metric, F.Cu at (230.8, 92.1)
- added C21: 4u7, Capacitor_SMD:C_1206_3216Metric, F.Cu at (221.1, 95.6)
- added C7: 4u7, Capacitor_SMD:C_1206_3216Metric, F.Cu at (221.1, 78.9)
- added C8: 4u7, Capacitor_SMD:C_1206_3216Metric, F.Cu at (221.1, 82.2)
- added C9: 100n, Capacitor_SMD:C_1210_3225Metric, F.Cu at (230.8, 79.3)
- added J1: PROG, Connector_PinHeader_2.54mm:PinHeader_1x05_P2.54mm_Vertical, F.Cu at (235.9, 79.5)
- added R12: 4k7, Resistor_SMD:R_0603_1608Metric, F.Cu at (226.0, 91.0)
- added R13: 100R, Resistor_SMD:R_0805_2012Metric, F.Cu at (230.2, 95.7)
- added R14: 4k7, Resistor_SMD:R_0603_1608Metric, F.Cu at (226.0, 93.5)
- added R15: 100R, Resistor_SMD:R_0805_2012Metric, F.Cu at (230.2, 98.6)
- added R16: 4k7, Resistor_SMD:R_0603_1608Metric, F.Cu at (226.0, 96.0)
- added R17: 100R, Resistor_SMD:R_0805_2012Metric, F.Cu at (230.2, 101.6)
- added U1: STM32G071KBTx, Package_QFP:LQFP-32_7x7mm_P0.8mm, F.Cu at (239.3, 97.7)
- added U2: 1EDN7550B, Package_TO_SOT_SMD:SOT-23-6, F.Cu at (240.8, 87.7)
- added U5: LM2937IMP-3.3N, Package_TO_SOT_SMD:SOT-223-3_TabPin2, F.Cu at (243.2, 81.3)
- C1, C4, C5, C6: footprint Capacitor_SMD:C_1206_3216Metric -> Capacitor_SMD:C_1210_3225Metric
Connections:
- net Net-(Q1-G) renamed /MDR
- C2 pad 1: /OUT -> /SENSE
- D1 pad 2: /OUT -> /SENSE

Commit message: PCB v1
Parts:
- removed D2: LED, Resistor_SMD:R_0603_1608Metric
- added C22: 100u, Capacitor_THT:CP_Radial_D10.0mm_P5.00mm, F.Cu at (233.9, 28.4)
- added C23: 4u7, Capacitor_SMD:C_1206_3216Metric, F.Cu at (186.0, 56.6)
- added C24: 4u7, Capacitor_SMD:C_1206_3216Metric, F.Cu at (188.4, 56.6)
- added C25: 100u, Capacitor_THT:CP_Radial_D10.0mm_P5.00mm, F.Cu at (192.9, 28.4)
- added C26: 100n/50V, Capacitor_SMD:C_0603_1608Metric, F.Cu at (144.8, 39.8)
- added C27: 100n, Capacitor_SMD:C_0603_1608Metric, F.Cu at (172.1, 58.2)
- added C28: 10p, Capacitor_SMD:C_0603_1608Metric, B.Cu at (263.8, 19.5)
- added C29: 1u/50V, Capacitor_SMD:C_0603_1608Metric, B.Cu at (152.4, 35.6)
- added C30: 4u7, Capacitor_SMD:C_1206_3216Metric, F.Cu at (153.0, 20.8)
- added C31: 1u/50V, Capacitor_SMD:C_0603_1608Metric, B.Cu at (153.0, 30.8)
- added C32: 1u/50V, Capacitor_SMD:C_0603_1608Metric, B.Cu at (149.2, 35.6)
- added C33: 1u/50V, Capacitor_SMD:C_0603_1608Metric, B.Cu at (150.8, 35.6)
- added D10: BAT46GWX, Diode_SMD:D_SOD-123, B.Cu at (148.8, 30.6)
- added D11: ESDA25P35, Diode_SMD:D_0603_1608Metric, F.Cu at (160.6, 23.4)
- added D12: ESDA25W, pulsarLib:SOT-323L, F.Cu at (154.2, 39.9)
- added D3: SK86, Diode_SMD:D_SMC, F.Cu at (237.5, 48.5)
- added D4: LED_CV, LED_SMD:LED_0603_1608Metric, F.Cu at (207.4, 59.4)
- added D5: OUT, LED_SMD:LED_0603_1608Metric, F.Cu at (262.1, 63.2)
- added D6: LED_CC, LED_SMD:LED_0603_1608Metric, F.Cu at (200.2, 59.4)
- added D7: SK86, Diode_SMD:D_SMC, F.Cu at (237.5, 41.5)
- added D8: PWR, LED_SMD:LED_0603_1608Metric, F.Cu at (183.8, 60.8)
- added D9: ESDA25P35, Diode_SMD:D_0603_1608Metric, B.Cu at (153.2, 20.6)
- added DI1: SSD1306, pulsarLib:SSD1306, F.Cu at (169.0, 32.5)
- added F1: Fuse, Fuse:Fuse_1206_3216Metric, F.Cu at (186.5, 41.0)
- added J3: Barrel_Jack_Switch, Connector_BarrelJack:BarrelJack_Horizontal, F.Cu at (158.4, 59.4)
- added J4: SCREW, pulsarLib:DEGSON DG301-5.0-2.0P, F.Cu at (147.7, 51.3)
- added J5: BANANA, pulsarLib:BANANA 4mm, F.Cu at (259.2, 40.2)
- added J6: SCREW, pulsarLib:DEGSON DG301-5.0-2.0P, F.Cu at (263.0, 23.5)
- added J7: UBC-RA-TF (HF), pulsarLib:UBC-RA-TF (HF), F.Cu at (150.2, 23.8)
- added L1: 33uH, pulsarLib:DPO-5.0-33, F.Cu at (217.5, 45.0)
- added Logo1: ~, pulsarLib:Bart's Design, F.Cu at (192.6, 19.2)
- added Logo2: ~, pulsarLib:PULSAR, F.Cu at (221.6, 25.2)
- added Q2: IRFR5305TRL, Package_TO_SOT_SMD:TO-252-2, F.Cu at (198.0, 40.7)
- added Q3: AOD2910, Package_TO_SOT_SMD:TO-252-2, F.Cu at (198.0, 49.5)
- added Q4: BC-817-16-DIO, Package_TO_SOT_SMD:SOT-23, F.Cu at (180.1, 49.0)
- added Q5: STL6P3LLH6, pulsarLib:PowerFLAT 3.3x3.3, B.Cu at (144.4, 37.6)
- added R10: 5k1, Resistor_SMD:R_0603_1608Metric, B.Cu at (155.6, 32.4)
- added R11: 10k, Resistor_SMD:R_0603_1608Metric, F.Cu at (169.6, 45.0)
- added R18: R, Resistor_SMD:R_0603_1608Metric, B.Cu at (256.8, 64.5)
- added R19: 1k, Resistor_SMD:R_0603_1608Metric, F.Cu at (190.7, 39.5)
- added R20: 1k, Resistor_SMD:R_0603_1608Metric, F.Cu at (190.5, 49.5)
- added R21: 22k, Resistor_SMD:R_0603_1608Metric, B.Cu at (179.3, 56.0)
- added R22: 22k, Resistor_SMD:R_0603_1608Metric, B.Cu at (178.8, 53.0)
- added R23: 4R7, Resistor_SMD:R_1206_3216Metric, F.Cu at (187.0, 49.0)
- added R24: 4R7, Resistor_SMD:R_1206_3216Metric, F.Cu at (187.0, 46.5)
- added R25: 10k, Resistor_SMD:R_0603_1608Metric, B.Cu at (176.3, 33.0)
- added R26: 1k, Resistor_SMD:R_0603_1608Metric, F.Cu at (177.2, 49.0)
- added R27: 10k, Resistor_SMD:R_0603_1608Metric, F.Cu at (169.8, 57.4)
- added R28: 1k, Resistor_SMD:R_0603_1608Metric, F.Cu at (169.8, 59.0)
- added R29: 1k, Resistor_SMD:R_0603_1608Metric, B.Cu at (200.2, 57.6)
- added R3: 8m, Resistor_SMD:R_2512_6332Metric, F.Cu at (237.0, 34.5)
- added R30: 4k7, Resistor_SMD:R_0603_1608Metric, B.Cu at (175.8, 20.0)
- added R31: 4k7, Resistor_SMD:R_0603_1608Metric, B.Cu at (162.4, 19.8)
- added R32: 10k, Resistor_SMD:R_0603_1608Metric, B.Cu at (164.8, 52.4)
- added R33: 22k, Resistor_SMD:R_0603_1608Metric, F.Cu at (263.0, 20.0)
- added R34: 1k, Resistor_SMD:R_0603_1608Metric, F.Cu at (263.0, 18.5)
- added R35: 1k, Resistor_SMD:R_0603_1608Metric, B.Cu at (207.4, 57.6)
- added R36: 1k, Resistor_SMD:R_0603_1608Metric, B.Cu at (179.8, 61.4)
- added R37: R, Resistor_SMD:R_0603_1608Metric, B.Cu at (173.5, 37.5)
- added R38: R, Resistor_SMD:R_0603_1608Metric, B.Cu at (172.5, 33.5)
- added R39: 5k1, Resistor_SMD:R_0603_1608Metric, B.Cu at (149.0, 23.6)
- added R4: 4R7, Resistor_SMD:R_1206_3216Metric, F.Cu at (180.5, 38.5)
- added R40: 10k, Resistor_SMD:R_0603_1608Metric, F.Cu at (161.8, 43.2)
- added R41: 4k7, Resistor_SMD:R_0603_1608Metric, F.Cu at (158.2, 50.8)
- added R42: 4k7, Resistor_SMD:R_0603_1608Metric, F.Cu at (159.8, 50.8)
- added R43: 4k7, Resistor_SMD:R_0603_1608Metric, F.Cu at (163.4, 43.2)
- added R44: 100k, Resistor_SMD:R_0603_1608Metric, B.Cu at (151.6, 50.0)
- added R45: 100k, Resistor_SMD:R_0603_1608Metric, B.Cu at (151.6, 48.4)
- added R46: (NM), Resistor_SMD:R_0603_1608Metric, B.Cu at (151.6, 51.6)
- added R47: (NM), Resistor_SMD:R_0603_1608Metric, B.Cu at (151.6, 53.2)
- added R48: 100k, Resistor_SMD:R_0603_1608Metric, F.Cu at (146.2, 33.6)
- added R49: 100R, Resistor_SMD:R_0805_2012Metric, F.Cu at (144.8, 36.4)
- added R5: 4R7, Resistor_SMD:R_1206_3216Metric, F.Cu at (180.5, 36.0)
- added R50: 22k, Resistor_SMD:R_0603_1608Metric, B.Cu at (145.2, 42.0)
- added R51: 1k, Resistor_SMD:R_0603_1608Metric, B.Cu at (150.4, 46.0)
- added R52: 470R, Resistor_SMD:R_0603_1608Metric, F.Cu at (149.0, 31.8)
- added R53: 1k, Resistor_SMD:R_0603_1608Metric, F.Cu at (150.6, 31.8)
- added R6: 22k, Resistor_SMD:R_0603_1608Metric, F.Cu at (176.5, 29.0)
- added R7: 22k, Resistor_SMD:R_0603_1608Metric, B.Cu at (183.5, 29.5)
- added R8: 22k, Resistor_SMD:R_0603_1608Metric, F.Cu at (258.0, 18.5)
- added R9: 1k, Resistor_SMD:R_0603_1608Metric, F.Cu at (258.0, 20.0)
- added SW1: UP, Button_Switch_THT:SW_PUSH_6mm, F.Cu at (230.6, 64.9)
- added SW2: DOWN, Button_Switch_THT:SW_PUSH_6mm, F.Cu at (240.6, 64.9)
- added SW3: OK, Button_Switch_THT:SW_PUSH_6mm, F.Cu at (250.6, 64.9)
- added U3: 1EDN7550B, Package_TO_SOT_SMD:SOT-23-6, F.Cu at (182.4, 53.0)
- added U4: INA181A2IDBVR / INA169NA, Package_TO_SOT_SMD:SOT-23-6, F.Cu at (173.5, 26.5)
- added U6: STUSB4500QTR, Package_DFN_QFN:QFN-24-1EP_4x4mm_P0.5mm_EP2.7x2.7mm, B.Cu at (149.6, 39.9)
- C1: value 10u -> 1m; footprint Capacitor_SMD:C_1210_3225Metric -> Capacitor_THT:CP_Radial_D12.5mm_P5.00mm
- C10: footprint Capacitor_SMD:C_1210_3225Metric -> Capacitor_SMD:C_0603_1608Metric; moved to B.Cu
- C11, C12, C13, C16, C17, C18, C7, C8, R12, R13, R14, R15, R16, R17, U1: moved to B.Cu
- C14, C15: footprint Capacitor_SMD:C_1206_3216Metric -> Capacitor_SMD:C_0603_1608Metric
- C19, C20: footprint Capacitor_SMD:C_1210_3225Metric -> Capacitor_SMD:C_0603_1608Metric
- C2: value 100u -> 1m; footprint Capacitor_THT:CP_Radial_D10.0mm_P5.00mm -> Capacitor_THT:CP_Radial_D12.5mm_P5.00mm
- C3: value 100u -> 10u; footprint Capacitor_THT:CP_Radial_D10.0mm_P5.00mm -> Capacitor_SMD:C_1206_3216Metric
- C4: footprint Capacitor_SMD:C_1210_3225Metric -> Capacitor_SMD:C_1206_3216Metric
- C5, C6: value 10u -> C; footprint Capacitor_SMD:C_1210_3225Metric -> Capacitor_SMD:C_0603_1608Metric
- C9: value 100n -> 10p; footprint Capacitor_SMD:C_1210_3225Metric -> Capacitor_SMD:C_0603_1608Metric
- D1: value B2D06065E1 -> ESDA25P35; footprint Package_TO_SOT_SMD:TO-252-2 -> Diode_SMD:D_0603_1608Metric; moved to B.Cu
- Q1: value IRLR3110Z -> STL6P3LLH6; footprint Package_TO_SOT_SMD:TO-252-2 -> pulsarLib:PowerFLAT 3.3x3.3; moved to B.Cu
- R1: value R -> 10k(INA186)
- R2: value 10k -> 0R; footprint Resistor_SMD:R_0603_1608Metric -> Diode_SMD:D_0603_1608Metric; moved to B.Cu
- moved R2 97.9 mm to (144.9, 23.6), turned to 180 degrees
- moved C21 96.0 mm to (155.5, 25.5)
- moved C19 95.7 mm to (156.5, 27.5), turned to 180 degrees
- moved U5 94.8 mm to (161.0, 34.0)
- moved C20 93.9 mm to (155.6, 35.8), turned to 90 degrees
- moved D1 89.1 mm to (259.5, 26.0), turned to -90 degrees
- moved U1 86.4 mm to (169.3, 47.0), turned to -90 degrees
- moved U2 83.1 mm to (180.0, 31.0), turned to -90 degrees
- moved C15 83.0 mm to (168.2, 28.4), turned to -90 degrees
- moved C14 81.5 mm to (166.6, 28.4), turned to -90 degrees
- moved C10 79.5 mm to (168.5, 34.2)
- moved C3 75.6 mm to (186.0, 31.0), turned to 90 degrees
- moved J1 75.0 mm to (162.4, 64.6), turned to 90 degrees
- moved R1 74.8 mm to (176.5, 26.5), turned to 90 degrees
- moved C1 72.9 mm to (246.0, 28.5), turned to 90 degrees
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Connections:
- C1 pad 1: /CIN -> /SENSE
- C1 pad 2: /COUT -> GND
- C2 pad 1: /SENSE -> /CONV_INPUT
- C3 pad 1: /VCC -> /CONV_INPUT
- C4 pad 1: /CIN -> /SENSE
- C4 pad 2: /COUT -> GND
- C5 pad 1: /CIN -> GND
- C5 pad 2: /COUT -> /CURRENT_CMP
- C6 pad 1: /CIN -> GND
- C6 pad 2: /COUT -> /CURRENT
- D1 pad 1: unconnected-(D1-A-Pad1) -> /OUT
- D1 pad 2: /SENSE -> GND
- Q1 pad 1: /MDR -> Net-(U6-VDD)
- Q1 pad 2: /CIN -> Net-(U6-VDD)
- Q1 pad 3: GND -> Net-(U6-VDD)
- R1 pad 1: Net-(D2-K) -> /SENSE_OUT
- R2 pad 1: /MDR -> /USB_VBUS
- R2 pad 2: GND -> /VCC
- U1 pad 10: unconnected-(U1-PA3-Pad10) -> /CURRENT_CMP
- U1 pad 12: /PWM -> /CV_MODE
- U1 pad 13: unconnected-(U1-PA6-Pad13) -> /CC_MODE
- U1 pad 17: unconnected-(U1-PB2-Pad17) -> /IN_VOLTAGE
- U1 pad 18: unconnected-(U1-PA8-Pad18) -> /PWML
- U1 pad 19: unconnected-(U1-PA9/UCPD1_DBCC1-Pad19) -> /PWMH
- U1 pad 20: unconnected-(U1-PC6-Pad20) -> /PD_RST
- U1 pad 21: unconnected-(U1-PA10/UCPD1_DBCC2-Pad21) -> /PD_ALERT
- U1 pad 22: unconnected-(U1-PA11/PA9-Pad22) -> /PD_SCL
- U1 pad 23: unconnected-(U1-PA12/PA10-Pad23) -> /PD_SDA
- U1 pad 26: unconnected-(U1-PA15-Pad26) -> /BUTTON_L
- U1 pad 27: unconnected-(U1-PB3-Pad27) -> /BUTTON_M
- U1 pad 28: unconnected-(U1-PB4-Pad28) -> /BUTTON_R
- U1 pad 30: unconnected-(U1-PB6-Pad30) -> /SCL
- U1 pad 31: unconnected-(U1-PB7-Pad31) -> /SDA
- U1 pad 8: unconnected-(U1-PA1-Pad8) -> /VOLTAGE_CMP
Routing:
- net +3V3: track 0.00 -> 227.6 mm, vias 0 -> 11
- net /OUT: track 0.00 -> 157.3 mm
- net /VCC: track 0.00 -> 147.1 mm, vias 0 -> 13
- net /VOLTAGE_CMP: track 0.00 -> 121.3 mm, vias 0 -> 2
- net /SENSE: track 0.00 -> 113.3 mm
- net /BUTTON_R: track 0.00 -> 113.1 mm, vias 0 -> 1
- net /VOLTAGE: track 0.00 -> 113.0 mm, vias 0 -> 1
- net /BUTTON_M: track 0.00 -> 101.2 mm, vias 0 -> 1
- net /BUTTON_L: track 0.00 -> 88.3 mm, vias 0 -> 1
- net /L_OUT: track 0.00 -> 66.2 mm
- net /CV_MODE: track 0.00 -> 53.3 mm, vias 0 -> 1
- net /USB_VBUS: track 0.00 -> 47.5 mm, vias 0 -> 4
- net /CC_MODE: track 0.00 -> 43.0 mm, vias 0 -> 1
- net /L_IN: track 0.00 -> 38.9 mm
- net /SCL: track 0.00 -> 38.5 mm
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- added copper zone on F.Cu, net /CONV_INPUT
- added copper zone on B.Cu, net /HSW
- added copper zone on F.Cu, net /HSW
- added copper zone on F.Cu, net /LSW
- added copper zone on F.Cu, net /OUT
- added copper zone on F.Cu, net /SENSE
- added copper zone on B.Cu, net /VCC
- added copper zone on F.Cu, net /VCC
- added copper zone on B.Cu, net GND
- added copper zone on F.Cu, net GND
Other:
- board outline added: 127 x 51.2 mm
