File: pulsarPCB/pulsarPCB.kicad_sch (KiCad schematic)
At the start: 49 parts, among them Q1 IRLR3110Z, SW1 UP, SW2 DOWN, SW3 OK, U1 STM32G071KBTx, U2 1EDN7550B, U3 INA282AID, U5 LM2937IMP-3.3N

Commit message: change topology
Parts:
- removed U3: INA282AID, symbol Amplifier_Current:INA282
- added C22, C25: 100u, Capacitor_THT:CP_Radial_D10.0mm_P5.00mm, symbol Device:C_Polarized
- added C23, C24: 4u7, Capacitor_SMD:C_1206_3216Metric, symbol Device:C
- added C26: 100n, Capacitor_SMD:C_1210_3225Metric, symbol Device:C
- added D3, D4: B2D06065E1, Package_TO_SOT_SMD:TO-252-2, symbol Device:D_Schottky_AKA
- added D5: LED, Resistor_SMD:R_0603_1608Metric, symbol Device:LED
- added J1: PROG, Connector_PinHeader_2.54mm:PinHeader_1x05_P2.54mm_Vertical, symbol Connector_Generic:Conn_01x05
- added L1: 33uH, symbol Device:L
- added Q2: IRFR5305TRL, symbol Device:Q_PMOS_GDS
- added Q3: AOD2910, Package_TO_SOT_SMD:TO-252-2, symbol Device:Q_NMOS_GDS
- added R18: R, Resistor_SMD:R_0603_1608Metric, symbol Device:R
- added R19, R20, R21, R22: 1k, symbol Device:R
- added R23, R24: 4R7, symbol Device:R
- added U3: 1EDN7550B, Package_TO_SOT_SMD:SOT-23-6, symbol Driver_FET:1EDN7550B
- added U4: INA181A2IDBVR, Package_TO_SOT_SMD:SOT-23-6, symbol Amplifier_Current:INA181
- Q1: value IRLR3110Z -> AOD2910
- R3: value R -> 8m; Field4 (none) -> 0V04@5A
Connections:
- net +3V3: now also J1.1 (Pin_1), U4.6 (V+)
- net CURRENT: now also C26.1, U4.1
- net GND: now also C22.2, C23.1, C24.1, C25.2, C26.2, D3.3 (A), J1.3 (Pin_3), Q3.3 (S), R18.2, R20.2, R22.1, U3.2 (GND), U4.2 (GND), U4.5 (REF)
- net MDR: now also Q1.1 (G), R2.1; no longer R3.1, R4.2, R5.1
- net OUT: now also U4.4 (-)
- net PWM: no longer R6.1
- net SENSE: now also U4.3 (+)
- net VCC: now also C23.2, C24.2, C25.1, Q2.3 (S), R19.1, U3.4 (VDD)
- net SYS_RST: now reaches R11.2, U1.6 (PF2)
- net SYS_RST: now also J1.5 (Pin_5)
- net SYS_SWDIO: now reaches U1.24 (PA13)
- net SYS_SWDIO: now also J1.4 (Pin_4)
- net SYS_SWDCLK: now reaches U1.25 (PA14)
- net SYS_SWDCLK: now also J1.2 (Pin_2)
- new net: R24.2, U3.6 (OUT_SNK)
- new net: D3.2 (K), L1.1, Q2.2 (D)
- new net: D4.3 (A), L1.2, Q3.2 (D)
- new net: D5.1 (K), R18.1
- new net: D5.2 (A), R3.2
- new net: R22.2, U3.1 (IN-)
- new net: R21.2, U3.3 (IN+)
- new net: C22.1, D4.2 (K), R3.1
- new net: R23.1, U3.5 (OUT_SRC)
- new net HSW: Q2.1 (G), R19.2, R23.2, R24.1
- new net LSW: Q3.1 (G), R20.1, R4.2, R5.1
- new net PWMH: R21.1
- new net PWML: R6.1
Other:
- moved on the sheet: C1, C10, C11, C12, C13, C14, C15, C16, C17, C18, C2, C3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

Commit message: PCB v1
Parts:
- removed C1: 10u, Capacitor_SMD:C_1210_3225Metric, symbol Device:C
- removed C26: 100n, Capacitor_SMD:C_1210_3225Metric, symbol Device:C
- removed C3: 100u, Capacitor_THT:CP_Radial_D10.0mm_P5.00mm, symbol Device:C_Polarized
- removed D1, D3, D4: B2D06065E1, Package_TO_SOT_SMD:TO-252-2, symbol Device:D_Schottky_AKA
- removed D2: LED, Resistor_SMD:R_0603_1608Metric, symbol Device:LED
- removed Q1: AOD2910, Package_TO_SOT_SMD:TO-252-2, symbol Device:Q_NMOS_GDS
- removed T1: ~, symbol pulsarLib:transformer-2part
- added C1: 1m, Capacitor_THT:CP_Radial_D12.5mm_P5.00mm, symbol Device:C_Polarized
- added C27: 100n, Capacitor_SMD:C_0603_1608Metric, symbol Device:C
- added C28: 10p, Capacitor_SMD:C_0603_1608Metric, symbol Device:C
- added C3: 10u, Capacitor_SMD:C_1206_3216Metric, symbol Device:C
- added D1: ESDA25P35, Diode_SMD:D_0603_1608Metric, symbol Device:D_Zener
- added D3, D7: SK86, Diode_SMD:D_SMC, symbol Device:D_Schottky
- added D4: LED_CV, LED_SMD:LED_0603_1608Metric, symbol Device:LED
- added D6: LED_CC, LED_SMD:LED_0603_1608Metric, symbol Device:LED
- added D8: PWR, LED_SMD:LED_0603_1608Metric, symbol Device:LED
- added DI1: SSD1306, pulsarLib:SSD1306, symbol pulsarLib:SSD1306
- added F1: Fuse, Fuse:Fuse_1206_3216Metric, symbol Device:Fuse
- added J3: Barrel_Jack_Switch, Connector_BarrelJack:BarrelJack_Horizontal, symbol Connector:Barrel_Jack_Switch
- added J4, J6: SCREW, pulsarLib:DEGSON DG301-5.0-2.0P, symbol Connector_Generic:Conn_01x02
- added J5: BANANA, pulsarLib:BANANA 4mm, symbol Connector_Generic:Conn_01x02
- added J7: UBC-RA-TF (HF), pulsarLib:UBC-RA-TF (HF), symbol Connector:USB_C_Receptacle_USB2.0_16P
- added Logo1: ~, pulsarLib:Bart's Design, symbol pulsarLib:Bart's_Design
- added Logo2: ~, pulsarLib:PULSAR, symbol pulsarLib:PULSAR
- added Q4: BC-817-16-DIO, Package_TO_SOT_SMD:SOT-23, symbol Device:Q_NPN_BEC
- added R25, R27, R32: 10k, Resistor_SMD:R_0603_1608Metric, symbol Device:R
- added R26, R28, R29, R34, R35, R36: 1k, Resistor_SMD:R_0603_1608Metric, symbol Device:R
- added R30, R31: 4k7, Resistor_SMD:R_0603_1608Metric, symbol Device:R
- added R33: 22k, Resistor_SMD:R_0603_1608Metric, symbol Device:R
- added R37, R38: R, Resistor_SMD:R_0603_1608Metric, symbol Device:R
- added R39: 5k1, Resistor_SMD:R_0603_1608Metric, symbol Device:R
- C10, C19, C20: footprint Capacitor_SMD:C_1210_3225Metric -> Capacitor_SMD:C_0603_1608Metric
- C14, C15: footprint Capacitor_SMD:C_1206_3216Metric -> Capacitor_SMD:C_0603_1608Metric
- C2: value 100u -> 1m; footprint Capacitor_THT:CP_Radial_D10.0mm_P5.00mm -> Capacitor_THT:CP_Radial_D12.5mm_P5.00mm; Field4 EEUFC1J101 -> EEUFR1V102
- C4: footprint Capacitor_SMD:C_1210_3225Metric -> Capacitor_SMD:C_1206_3216Metric
- C5, C6: value 10u -> C; footprint Capacitor_SMD:C_1210_3225Metric -> Capacitor_SMD:C_0603_1608Metric
- C9: value 100n -> 10p; footprint Capacitor_SMD:C_1210_3225Metric -> Capacitor_SMD:C_0603_1608Metric
- D5: value LED -> OUT; footprint Resistor_SMD:R_0603_1608Metric -> LED_SMD:LED_0603_1608Metric
- L1: footprint (none) -> pulsarLib:DPO-5.0-33; Field4 (none) -> DPO-5.0-33
- Q2: footprint (none) -> Package_TO_SOT_SMD:TO-252-2
- R1: value R -> 10k(INA186)
- R10: value 8m -> 5k1; footprint (none) -> Resistor_SMD:R_0603_1608Metric
- R11, R19, R20, R9: footprint (none) -> Resistor_SMD:R_0603_1608Metric
- R2: value 10k -> 0R; footprint Resistor_SMD:R_0603_1608Metric -> Diode_SMD:D_0603_1608Metric; Field5 (none) -> Mount only if PD IC isn't fitted
- R21, R22, R6, R7: value 1k -> 22k; footprint (none) -> Resistor_SMD:R_0603_1608Metric
- R23, R24, R4, R5: footprint (none) -> Resistor_SMD:R_1206_3216Metric
- R3: footprint (none) -> Resistor_SMD:R_2512_6332Metric
- R8: value 22 -> 22k; footprint (none) -> Resistor_SMD:R_0603_1608Metric
- SW1, SW2, SW3: footprint (none) -> Button_Switch_THT:SW_PUSH_6mm
- U4: value INA181A2IDBVR -> INA181A2IDBVR / INA169NA
Connections:
- net +3V3: now also D8.2 (A), DI1.2 (VCC), R30.1, R31.1
- net BUTTON_L: now also U1.26 (PA15)
- net BUTTON_M: now also U1.27 (PB3)
- net BUTTON_R: now also U1.28 (PB4)
- net CURRENT: now also C6.2, R38.2; no longer U4.1
- net GND: now also C4.2, C5.1, C6.1, R10.2, C1.2, C27.2, C28.2, C3.2, D1.2 (A), D3.2 (A), DI1.1 (GND), J3.2, J4.1 (Pin_1), J5.2 (Pin_2), J6.2 (Pin_2), J7.A1 (GND), J7.A12 (GND), J7.B1 (GND), J7.B12 (GND), J7.S1 (SHIELD), Q4.2 (E), R28.2, R29.2, R32.2, R34.2, R35.2, R36.2, R39.2; no longer R2.2
- net HSW: now also R4.2, R5.1; no longer R23.2, R24.1
- net LSW: now also R23.2, R24.1; no longer R4.2, R5.1
- net OUT: now also D5.2 (A), R3.2, D1.1 (K), J5.1 (Pin_1), J6.1 (Pin_1), R33.1; no longer R10.2
- net PWMH: now also U1.19 (PA9/UCPD1_DBCC1), R26.1; no longer R21.1
- net PWML: now also R21.1, U1.18 (PA8); no longer R6.1
- net SENSE: now also C22.1, C4.1, R3.1, C1.1, D7.1 (K); no longer C2.1, R10.1
- net SYS_SWDCLK: now also R32.1
- net VCC: now also R2.2, F1.1, J3.1, J4.2 (Pin_2), R25.1, R27.1; no longer C25.1, Q2.3 (S), R19.1
- net L_IN: now reaches L1.1, Q2.2 (D)
- net L_IN: now also D3.1 (K)
- net L_OUT: now reaches L1.2, Q3.2 (D)
- net L_OUT: now also D7.2 (A)
- net SENSE_OUT: now reaches R1.1
- net SENSE_OUT: now also U4.1, R37.1, R38.1
- net CURRENT_CMP: now reaches U1.10 (PA3)
- net CURRENT_CMP: now also C5.2, R37.2
- net CC_MODE: now reaches U1.13 (PA6)
- net CC_MODE: now also D6.2 (A)
- net IN_VOLTAGE: now reaches U1.17 (PB2)
- net IN_VOLTAGE: now also C27.1, R27.2, R28.1
- net PD_RST: now reaches U1.20 (PC6)
- net PD_ALERT: now reaches U1.21 (PA10/UCPD1_DBCC2)
- net PD_SCL: now reaches U1.22 (PA11/PA9)
- net PD_SDA: now reaches U1.23 (PA12/PA10)
- net SCL: now reaches U1.30 (PB6)
- net SCL: now also DI1.3 (SCL), R31.2
- net SDA: now reaches U1.31 (PB7)
- net SDA: now also DI1.4 (SDA), R30.2
- net VOLTAGE_CMP: now reaches U1.8 (PA1)
- net VOLTAGE_CMP: now also C28.1, R33.2, R34.1
- removed net CIN: C4.1, C5.1, C6.1
- removed net COUT: C4.2, C5.2, C6.2
- net MDR renamed USB_VBUS
- net USB_VBUS: now also J7.A4 (VBUS), J7.A9 (VBUS), J7.B4 (VBUS), J7.B9 (VBUS)
- net PWM renamed CV_MODE
- net CV_MODE: now also D4.2 (A)
- new net: Q4.1 (B), R26.2
- new net: D8.1 (K), R36.1
- new net: D4.1 (K), R35.1
- new net: Q4.3 (C), R25.2, R6.1
- new net: D6.1 (K), R29.1
- new net CC1: J7.A5 (CC1), R10.1
- new net CC2: J7.B5 (CC2), R39.1
- new net CONV_INPUT: C2.1, C25.1, C3.1, F1.2, Q2.3 (S), R19.1
- no-connect marks 27 -> 16
Other:
- added sheet POWER_DELIVERY (PD.kicad_sch)
- note added: "3300mV/11(div) = 36300mV 36300mV/4095 steps = 8,9mV/step"
- note added: "3300mv*23(divider) = 75900mV 75900mV/4095 steps = 18,5mV/step"
- note added: "IN: 5-20V OUT U: max 20/30V(due to opamp variant) OUT I: max 5A POWER: max 50W"
- note added: "INA181: 3300mV/50(opamp gain) = 66mV 66mV/0,008R(shunt) = 8250mA(max current) 8250mA/4095 = 2mA/step"
- note added: "^CLASSIC POWER_DELIVERY^"
- note removed: "0V04@5A"
- note removed: "IN: 5-20V OUT U: max 60V OUT I: max 5A POWER: max 50W"
- note removed: "IN: 58V OUT: 2V52 ADC: 3127 step @ 58V 54 step / V 18,6mV / step"
- note removed: "in: 0V04 @ 5A out: 2V @ 5A ADC: 2482 step @ 5A 496 step / A 2mA/step"
- moved on the sheet: C10, C11, C12, C13, C14, C15, C16, C17, C18, C19, C20, C21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
